File: PacketRadio/PacketRadio.kicad_pcb (KiCad board)
At the start: 2 copper layers, 53.2 x 47 mm, 63 parts, among them J1 AudioJack3_Ground, J4 UART Connector, J5 USB_B_Micro, J6 Kenwood Connector, Q1 BC847, Q2 BC857, U1 PCM2912APJT, U2 FT232RL, U3 XR22404CG28-F, Y1 6 MHz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

Commit message: Update first draft
Parts:
- removed C28: 150 uF, Capacitor_SMD:C_1206_3216Metric_Pad1.42x1.75mm_HandSolder
- removed J1: AudioJack3_Ground, Connector_Audio:Jack_3.5mm_CUI_SJ1-3533NG_Horizontal
- removed J4: UART Connector, Connector_PinHeader_1.00mm:PinHeader_1x05_P1.00mm_Vertical
- removed J6: Kenwood Connector, TerminalBlock_Phoenix:TerminalBlock_Phoenix_MKDS-1,5-4_1x04_P5.00mm_Horizontal
- added D1: D, Diode_SMD:D_0603_1608Metric_Pad1.05x0.95mm_HandSolder, F.Cu at (246.0, 101.9)
- added FL1: EMI_Filter_CommonMode, ACM2012-201-2P-T001:FIL_ACM2012-201-2P-T001, F.Cu at (248.1, 97.6)
- added GND +5V RX TX: UART Connector, Connector_PinHeader_1.00mm:PinHeader_1x04_P1.00mm_Vertical, F.Cu at (232.7, 72.4)
- added Left: Left, TestPoint:TestPoint_Pad_D3.0mm, F.Cu at (205.7, 73.5)
- added MIC: MIC, TestPoint:TestPoint_Pad_D3.0mm, F.Cu at (216.2, 84.5)
- added MIC GND: MIC_GND, TestPoint:TestPoint_Pad_D3.0mm, F.Cu at (216.2, 95.5)
- added R15: 0, Resistor_SMD:R_0603_1608Metric_Pad1.05x0.95mm_HandSolder, F.Cu at (222.2, 86.0)
- added REF**: OSHW-Logo2_14.6x12mm_SilkScreen, Symbol:OSHW-Logo2_14.6x12mm_SilkScreen, B.Cu at (207.7, 77.5)
- added Right: Right, TestPoint:TestPoint_Pad_D3.0mm, F.Cu at (205.7, 79.1)
- added SP: SP, TestPoint:TestPoint_Pad_D3.0mm, F.Cu at (216.2, 90.0)
- added SP GND: SP_GND, TestPoint:TestPoint_Pad_D3.0mm, F.Cu at (216.2, 101.0)
- C12, C13, C7, Q1, Q2, R17, R20: moved to B.Cu
- C26: footprint Capacitor_SMD:C_1206_3216Metric_Pad1.42x1.75mm_HandSolder -> Capacitor_SMD:C_0603_1608Metric_Pad1.05x0.95mm_HandSolder
- L1: moved to F.Cu
- U3: footprint XR22404CG28-F:SOP65P780X200-28N -> Package_SO:SSOP-28_5.3x10.2mm_P0.65mm
- Y1, Y3: footprint Crystal:Crystal_SMD_HC49-SD_HandSoldering -> Crystal:Crystal_HC49-4H_Vertical
- moved H1 76.0 mm to (200.7, 101.5)
- moved H2 58.4 mm to (200.7, 73.5)
- moved H4 56.3 mm to (252.7, 101.5)
- moved H3 35.8 mm to (252.7, 73.5)
- moved C6 30.0 mm to (230.5, 86.0), turned to 270 degrees
- moved Y1 27.3 mm to (227.7, 79.6), turned to 270 degrees
- moved R1 26.9 mm to (230.5, 82.0), turned to 90 degrees
- moved C4 26.0 mm to (230.5, 78.0), turned to 270 degrees
- moved Y3 25.2 mm to (233.7, 84.5)
- moved C22 24.7 mm to (252.5, 80.0), turned to 180 degrees
- moved C26 23.7 mm to (252.6, 77.5), turned to 180 degrees
- moved R17 21.7 mm to (216.4, 78.0), turned to 90 degrees
- moved Q1 21.6 mm to (219.1, 77.9)
- moved C16 20.0 mm to (246.7, 79.7), turned to 0 degrees
- moved R13 16.1 mm to (243.8, 90.5)
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Connections:
- C2 pad 2: /SP -> Net-(C2-Pad2)
- F1 pad 1: Net-(C19-Pad1) -> Net-(D1-Pad2)
- J5 pad 2: (no net) -> Net-(FL1-Pad3)
- J5 pad 3: (no net) -> Net-(FL1-Pad1)
- U3 pad 15: (no net) -> USB_N
- U3 pad 16: (no net) -> USB_P
Routing:
- net VDDA33-10: track 73.9 -> 0.00 mm
- net VDD33-15: track 53.4 -> 0.00 mm
- net /SP: track 56.9 -> 8.73 mm
- net BGND: track 41.3 -> 2.67 mm, vias 5 -> 1
- net Net-(C15-Pad2): track 48.3 -> 14.4 mm
- net MIC: track 10.4 -> 36.5 mm
- net VBUS: track 107.9 -> 85.4 mm, vias 1 -> 0
- net VCC33: track 0.00 -> 22.4 mm, vias 0 -> 1
- net Net-(C14-Pad2): track 31.6 -> 14.3 mm
- net USB_FT_N: track 0.00 -> 14.8 mm
- net USB_FT_P: track 0.65 -> 14.2 mm
- net (no net): track 13.2 -> 0.00 mm
- net XTI: track 33.0 -> 20.6 mm, vias 0 -> 1
- net RTS: track 13.2 -> 25.3 mm, vias 0 -> 1
- net XTO: track 30.6 -> 19.1 mm, vias 0 -> 1
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Other:
- board size 53.2 x 47 mm -> 58 x 34 mm
- board text added: "DO2FMW"
- board text added: "Packet Radio Revision 1 - 02/2019 github.com/elnappo/PCB"
